File: episodes/002-jordan-pilot-episode/5-electronics/gamer-companion.kicad_sch (KiCad schematic)
At the start: 46 parts, among them J1 USB harness, J2 BLOWER, J3 SPEAKER, Q1 AO3400A, U1 AP2112K-3.3TRG1, U2 ESP32-S3-WROOM-1-N16R8, U3 MAX98357AETE+T, U4 ICS-43434, U5 AM312

Commit message: 002 stage 5: routed 2-layer board, DRC clean
ESP32-S3-WROOM-1 on a vertical board behind the face: PIR and eye LEDs
on the front, module, LDO, amp, mic and connectors on the back.
ERC 0, DRC 0 violations / 0 unconnected.

KiCad kit: BOTTOM (parts on the bottom face), per-face NO_PARTS,
TRIM_COURTYARD for modules with oversized antenna courtyards,
PREROUTE starting on bottom pads. Episode 001 places identically.

Co-Authored-By: Claude Opus 5.5 <noreply@anthropic.com>
Parts:
- removed C2: 10uF, Capacitor_SMD:C_0805_2012Metric, symbol Device:C
- removed R2: 10k, Resistor_SMD:R_0603_1608Metric, symbol Device:R
- removed TP1: VBUS, TestPoint:TestPoint_Pad_D1.5mm, symbol Connector:TestPoint
- removed TP2: 3V3, TestPoint:TestPoint_Pad_D1.5mm, symbol Connector:TestPoint
- removed TP3: GND, TestPoint:TestPoint_Pad_D1.5mm, symbol Connector:TestPoint
Connections:
- net AMP_SD: now also U2.12 (IO8); no longer U2.10 (IO17)
- net FAN_PWM: now also U2.20 (IO12); no longer U2.6 (IO6)
- net I2S_BCLK: now also U2.4 (IO4); no longer U2.7 (IO7)
- net I2S_DIN: now also U2.11 (IO18); no longer U2.9 (IO16)
- net I2S_LRCLK: now also U2.5 (IO5); no longer U2.8 (IO15)
- net LED_IO: now also U2.9 (IO16); no longer U2.5 (IO5)
- net MIC_SCK: now also U2.17 (IO9); no longer U2.11 (IO18)
- net MIC_SD: now also U2.19 (IO11); no longer U2.17 (IO9)
- net MIC_WS: now also U2.18 (IO10); no longer U2.12 (IO8)
- net PIR_OUT: now also U2.8 (IO15); no longer U2.4 (IO4)
Other:
- note added: "MCU: ESP32-S3-WROOM-1-N16R8 on the board's back, antenna on the top edge (copper-free). Native USB on IO19/IO20 for flashing (no buttons needed). Pins picked for the layout: IO15 PIR (level with the PIR's OUT leg), IO16 LEDs, IO4/5/18 amp BCLK/LRCLK/DIN, IO8 amp SD, IO9/10/11 mic SCK/WS/SD, IO12 fan PWM. IO35-37 belong to the octal PSRAM."
- note removed: "MCU: ESP32-S3-WROOM-1-N16R8 on the board's back, antenna on the top edge (copper-free). Native USB on IO19/IO20 for flashing (no buttons needed). IO4 PIR, IO5 LEDs, IO6 fan PWM, IO7/15/16/17 amp I2S + SD, IO18/8/9 mic I2S. IO35-37 belong to the octal PSRAM."
